Commit message: Adds optional support for Xamla's rounded cap * implementing xamla_cap option in macro ur5_robot. * adding visual and collision meshes.

File: ur_description/urdf/ur5.urdf.xacro (robot description, xacro)
@@ -68,5 +68,13 @@
     </inertial>
   </xacro:macro>
-  <xacro:macro name="ur5_robot" params="prefix joint_limited">
+  <!--
+    The parameter xamla_cap enables optional support for Xamla's rounded cap (wrist 2),
+    increasing the collision free space.
+    If set, visual and collision meshes are loaded from the files provided in the following
+    repository: https://github.com/Xamla/xamla_egomo.
+    More information on the cap and the 3D-printable models can be found at:
+    https://github.com/Xamla/xamla_egomo/tree/master/egomo_3d_printed_parts/egomo-1
+  -->
+  <xacro:macro name="ur5_robot" params="prefix joint_limited xamla_cap:=false">
     <link name="${prefix}base_link" >
       <visual>
@@ -227,13 +235,23 @@
       <visual>
         <geometry>
-          <mesh filename="package://ur_description/meshes/ur5/visual/wrist2.dae" />
-        </geometry>
-        <material name="LightGrey">
-          <color rgba="0.7 0.7 0.7 1.0"/>
-        </material>
-      </visual>
-      <collision>
-        <geometry>
-          <mesh filename="package://ur_description/meshes/ur5/collision/wrist2.stl" />
+          <xacro:if value="${xamla_cap}">
+            <mesh filename="package://ur_description/meshes/ur5/visual/wrist2_rounded.dae" />
+          </xacro:if>
+          <xacro:unless value="${xamla_cap}">
+            <mesh filename="package://ur_description/meshes/ur5/visual/wrist2.dae" />
+          </xacro:unless>
+        </geometry>
+        <material name="LightGrey">
+          <color rgba="0.7 0.7 0.7 1.0"/>
+        </material>
+      </visual>
+      <collision>
+        <geometry>
+          <xacro:if value="${xamla_cap}">
+            <mesh filename="package://ur_description/meshes/ur5/collision/wrist2_rounded.stl" />
+          </xacro:if>
+          <xacro:unless value="${xamla_cap}">
+	    <mesh filename="package://ur_description/meshes/ur5/collision/wrist2.stl" />
+          </xacro:unless>
         </geometry>
       </collision>

Commit message: Setting joint limits to 'elbow up' for wall mount.

File: ur_description/urdf/ur5.urdf.xacro (robot description, xacro)
@@ -135,5 +135,5 @@
       </xacro:unless>
       <xacro:if value="${joint_limited}">
-        <limit lower="${-pi}" upper="${pi}" effort="150.0" velocity="3.15"/>
+        <limit lower="${-1.25 * pi}" upper="${0.25 * pi}" effort="150.0" velocity="3.15"/>
       </xacro:if>
       <dynamics damping="0.0" friction="0.0"/>
@@ -166,5 +166,5 @@
       </xacro:unless>
       <xacro:if value="${joint_limited}">
-        <limit lower="${-pi}" upper="${pi}" effort="150.0" velocity="3.15"/>
+        <limit lower="${-pi}" upper="0.0" effort="150.0" velocity="3.15"/>
       </xacro:if>
       <dynamics damping="0.0" friction="0.0"/>
@@ -224,10 +224,11 @@
       <origin xyz="0.0 ${wrist_1_length} 0.0" rpy="0.0 0.0 0.0" />
       <axis xyz="0 0 1" />
-      <xacro:unless value="${joint_limited}">
+      <!-- <xacro:unless value="${joint_limited}">
         <limit lower="${-2.0 * pi}" upper="${2.0 * pi}" effort="28.0" velocity="3.2"/>
       </xacro:unless>
       <xacro:if value="${joint_limited}">
         <limit lower="${-pi}" upper="${pi}" effort="28.0" velocity="3.2"/>
-      </xacro:if>
+      </xacro:if>-->
+	<limit lower="${-2.0 * pi}" upper="${2.0 * pi}" effort="28.0" velocity="3.2"/>
       <dynamics damping="0.0" friction="0.0"/>
     </joint>
@@ -265,10 +266,11 @@
       <origin xyz="0.0 0.0 ${wrist_2_length}" rpy="0.0 0.0 0.0" />
       <axis xyz="0 1 0" />
-      <xacro:unless value="${joint_limited}">
+      <!-- <xacro:unless value="${joint_limited}">
         <limit lower="${-2.0 * pi}" upper="${2.0 * pi}" effort="28.0" velocity="3.2"/>
       </xacro:unless>
       <xacro:if value="${joint_limited}">
         <limit lower="${-pi}" upper="${pi}" effort="28.0" velocity="3.2"/>
-      </xacro:if>
+      </xacro:if>-->
+	<limit lower="${-2.0 * pi}" upper="${2.0 * pi}" effort="28.0" velocity="3.2"/>
       <dynamics damping="0.0" friction="0.0"/>
     </joint>
